Commit message: Gazebo: diff drive, joint state publisher & laser scan rviz: visualize scanned mapped

File: urdf/vacuumcleaner/model.urdf (robot description, URDF)
Before this commit: robot vacuumcleaner, 4 links, 3 joints
Links:
- added link base_scan, mass 0.1; collision sphere radius=0.05; visual sphere radius=0.05
Joints:
- removed joint joint_left_wheel
- removed joint joint_right_wheel
- added joint lidar_sensor_joint: type fixed, parent base_link, child base_scan
- added joint wheel_left_joint: type continuous, parent base_link, child link_left_wheel, origin xyz=-0.05 -0.15 0 rpy=0 0 0, axis 0 1 0, limit effort=10000 velocity=1000
- added joint wheel_right_joint: type continuous, parent base_link, child link_right_wheel, origin xyz=-0.05 0.15 0 rpy=0 0 0, axis 0 1 0, limit effort=10000 velocity=1000

Commit message: update urdf to match dimensions of sdf

File: urdf/vacuumcleaner/model.urdf (robot description, URDF)
Before this commit: robot vacuumcleaner, 5 links, 4 joints
Links:
- link base_link: geometry collision box size=0.4 0.2 0.1; collision sphere radius=0.05
- link link_left_wheel: geometry collision cylinder length=0.05 radius=0.1; visual cylinder length=0.05 radius=0.1
- link link_right_wheel: geometry collision cylinder length=0.05 radius=0.1; visual cylinder length=0.05 radius=0.1
Joints:
- joint wheel_left_joint: origin xyz=-0.05 -0.15 0 rpy=0 0 0 -> xyz=0.1 0.13 0.1 rpy=0 0 0
- joint wheel_right_joint: origin xyz=-0.05 0.15 0 rpy=0 0 0 -> xyz=0.1 -0.13 0.1 rpy=0 0 0

Commit message: gazebo now uses urdf iso sdf

File: urdf/vacuumcleaner/model.urdf (robot description, URDF)
Before this commit: robot vacuumcleaner, 5 links, 4 joints
Links:
- removed link dummy
- removed link link_left_wheel
- removed link link_right_wheel
- link base_link: mass 5 -> 10; geometry collision box size=0.1 0.1 0.1; visual box size=0.1 0.1 0.1
- link base_scan: mass 0.1 -> 10
Joints:
- removed joint dummy_joint
- removed joint lidar_sensor_joint
- removed joint wheel_left_joint
- removed joint wheel_right_joint
- added joint base_scan_joint: type fixed, parent base_link, child base_scan, origin xyz=0 0 0.05

Commit message: Reworked urdf model

File: urdf/vacuumcleaner/model.urdf (robot description, URDF)
Before this commit: robot vacuumcleaner, 2 links, 1 joints
Links:
- added link base_footprint
- added link link_left_wheel, mass 0.2; collision cylinder length=0.04 radius=0.05; visual cylinder length=0.04 radius=0.05
- added link link_right_wheel, mass 0.2; collision cylinder length=0.04 radius=0.05; visual cylinder length=0.04 radius=0.05
- link base_link: mass 10 -> 5; geometry collision box size=0.4 0.15 0.1; collision sphere radius=0.01
- link base_scan: mass 10 -> 0.1
Joints:
- added joint base_joint: type fixed, parent base_footprint, child base_link, origin xyz=0 0 0 rpy=0 0 0
- added joint joint_left_wheel: type continuous, parent base_link, child link_left_wheel, origin xyz=-0.1 -0.10 -0.02 rpy=0 0 0, axis 0 1 0, limit effort=10000 velocity=1000
- added joint joint_right_wheel: type continuous, parent base_link, child link_right_wheel, origin xyz=-0.1 0.10 -0.02 rpy=0 0 0, axis 0 1 0, limit effort=10000 velocity=1000

Commit message: Navigation stack working tho trips up due to footprint not moving with robot

File: urdf/vacuumcleaner/model.urdf (robot description, URDF)
Before this commit: robot vacuumcleaner, 5 links, 4 joints
Joints:
- joint base_scan_joint: origin xyz=0 0 0.05 -> xyz=0 0 0.051

Commit message: changed urdf to look more like a vacuumcleaner bot iso stick with wheels

File: urdf/vacuumcleaner/model.urdf (robot description, URDF)
Before this commit: robot vacuumcleaner, 5 links, 4 joints
Links:
- link base_link: geometry collision cylinder length=0.04 radius=0.2; collision sphere radius=0.02
- link link_left_wheel: geometry collision cylinder length=0.02 radius=0.02; visual cylinder length=0.02 radius=0.02
- link link_right_wheel: geometry collision cylinder length=0.02 radius=0.02; visual cylinder length=0.02 radius=0.02
Joints:
- joint joint_left_wheel: origin xyz=-0.1 -0.10 -0.02 rpy=0 0 0 -> xyz=-0.1 -0.10 -0.04 rpy=0 0 0
- joint joint_right_wheel: origin xyz=-0.1 0.10 -0.02 rpy=0 0 0 -> xyz=-0.1 0.10 -0.04 rpy=0 0 0

Commit message: update rviz config with planners

File: urdf/vacuumcleaner/model.urdf (robot description, URDF)
Before this commit: robot vacuumcleaner, 5 links, 4 joints
Links:
- link link_left_wheel: geometry collision cylinder length=0.06 radius=0.02; visual cylinder length=0.06 radius=0.02
- link link_right_wheel: geometry collision cylinder length=0.06 radius=0.02; visual cylinder length=0.06 radius=0.02
Joints:
- joint joint_left_wheel: origin xyz=-0.1 -0.10 -0.04 rpy=0 0 0 -> xyz=-0.1 -0.10 -0.041 rpy=0 0 0
- joint joint_right_wheel: origin xyz=-0.1 0.10 -0.04 rpy=0 0 0 -> xyz=-0.1 0.10 -0.041 rpy=0 0 0

Commit message: Update inertia matrix

File: urdf/vacuumcleaner/model.urdf (robot description, URDF)
Before this commit: robot vacuumcleaner, 5 links, 4 joints
Links:
- link base_link: geometry collision cylinder length=0.04 radius=0.2; collision sphere radius=0.033
- link link_left_wheel: mass 0.2 -> 0.1; geometry collision cylinder length=0.018 radius=0.033; visual cylinder length=0.018 radius=0.033
- link link_right_wheel: mass 0.2 -> 0.1; geometry collision cylinder length=0.018 radius=0.033; visual cylinder length=0.018 radius=0.033
Joints:
- joint joint_left_wheel: origin xyz=-0.1 -0.10 -0.041 rpy=0 0 0 -> xyz=-0.1 -0.10 -0.054 rpy=0 0 0
- joint joint_right_wheel: origin xyz=-0.1 0.10 -0.041 rpy=0 0 0 -> xyz=-0.1 0.10 -0.054 rpy=0 0 0

Commit message: model now spins around z-axis

File: urdf/vacuumcleaner/model.urdf (robot description, URDF)
Before this commit: robot vacuumcleaner, 5 links, 4 joints
Links:
- link base_link: mass 5 -> 0.1
Joints:
- joint joint_left_wheel: limit effort=10000 velocity=1000 -> (none); origin xyz=-0.1 -0.10 -0.054 rpy=0 0 0 -> xyz=-0.02 -0.10 -0.054 rpy=0 0 0
- joint joint_right_wheel: limit effort=10000 velocity=1000 -> (none); origin xyz=-0.1 0.10 -0.054 rpy=0 0 0 -> xyz=-0.02 0.10 -0.054 rpy=0 0 0

Commit message: swap around left & right joint to make navigation work

File: urdf/vacuumcleaner/model.urdf (robot description, URDF)
Before this commit: robot vacuumcleaner, 5 links, 4 joints
Links:
- link base_link: mass 0.1 -> 2
Joints:
- joint joint_left_wheel: limit (none) -> effort=10000 velocity=1000; origin xyz=-0.02 -0.10 -0.054 rpy=0 0 0 -> xyz=-0.02 0.10 -0.054 rpy=0 0 0
- joint joint_right_wheel: limit (none) -> effort=10000 velocity=1000; origin xyz=-0.02 0.10 -0.054 rpy=0 0 0 -> xyz=-0.02 -0.10 -0.054 rpy=0 0 0
