Commit message: add nav2d exploration; robot stuck issue

File: src/vacuumcleaner/urdf/vacuumcleaner/model.urdf (robot description, URDF)
Before this commit: robot vacuumcleaner, 5 links, 4 joints
Links:
- removed link base_footprint
- removed link base_link
- removed link base_scan
- removed link link_left_wheel
- removed link link_right_wheel
- added link vacuumcleaner/base_footprint
- added link vacuumcleaner/base_link, mass 2; collision cylinder length=0.04 radius=0.2; collision sphere radius=0.033
- added link vacuumcleaner/base_scan, mass 0.1; collision sphere radius=0.05; visual sphere radius=0.05
- added link vacuumcleaner/link_left_wheel, mass 0.1; collision cylinder length=0.018 radius=0.033; visual cylinder length=0.018 radius=0.033
- added link vacuumcleaner/link_right_wheel, mass 0.1; collision cylinder length=0.018 radius=0.033; visual cylinder length=0.018 radius=0.033
Joints:
- removed joint base_joint
- removed joint base_scan_joint
- removed joint joint_left_wheel
- removed joint joint_right_wheel
- added joint vacuumcleaner/base_joint: type fixed, parent vacuumcleaner/base_footprint, child vacuumcleaner/base_link, origin xyz=0 0 0 rpy=0 0 0
- added joint vacuumcleaner/base_scan_joint: type fixed, parent vacuumcleaner/base_link, child vacuumcleaner/base_scan, origin xyz=0 0 0.051
- added joint vacuumcleaner/joint_left_wheel: type continuous, parent vacuumcleaner/base_link, child vacuumcleaner/link_left_wheel, origin xyz=-0.02 0.10 -0.054 rpy=0 0 0, axis 0 1 0, limit effort=10000 velocity=1000
- added joint vacuumcleaner/joint_right_wheel: type continuous, parent vacuumcleaner/base_link, child vacuumcleaner/link_right_wheel, origin xyz=-0.02 -0.10 -0.054 rpy=0 0 0, axis 0 1 0, limit effort=10000 velocity=1000

Commit message: get rid of vacuumcleaner/ prefix

File: src/vacuumcleaner/urdf/vacuumcleaner/model.urdf (robot description, URDF)
Before this commit: robot vacuumcleaner, 5 links, 4 joints
Links:
- removed link vacuumcleaner/base_footprint
- removed link vacuumcleaner/base_link
- removed link vacuumcleaner/base_scan
- removed link vacuumcleaner/link_left_wheel
- removed link vacuumcleaner/link_right_wheel
- added link base_footprint
- added link base_link, mass 2; collision cylinder length=0.04 radius=0.2; collision sphere radius=0.033
- added link base_scan, mass 0.1; collision sphere radius=0.05; visual sphere radius=0.05
- added link link_left_wheel, mass 0.1; collision cylinder length=0.018 radius=0.033; visual cylinder length=0.018 radius=0.033
- added link link_right_wheel, mass 0.1; collision cylinder length=0.018 radius=0.033; visual cylinder length=0.018 radius=0.033
Joints:
- removed joint vacuumcleaner/base_joint
- removed joint vacuumcleaner/base_scan_joint
- removed joint vacuumcleaner/joint_left_wheel
- removed joint vacuumcleaner/joint_right_wheel
- added joint base_joint: type fixed, parent base_footprint, child base_link, origin xyz=0 0 0 rpy=0 0 0
- added joint base_scan_joint: type fixed, parent base_link, child base_scan, origin xyz=0 0 0.051
- added joint joint_left_wheel: type continuous, parent base_link, child link_left_wheel, origin xyz=-0.02 0.10 -0.054 rpy=0 0 0, axis 0 1 0, limit effort=10000 velocity=1000
- added joint joint_right_wheel: type continuous, parent base_link, child link_right_wheel, origin xyz=-0.02 -0.10 -0.054 rpy=0 0 0, axis 0 1 0, limit effort=10000 velocity=1000

Commit message: Fixes robot stuck, but doesn't find route to explore

File: src/vacuumcleaner/urdf/vacuumcleaner/model.urdf (robot description, URDF)
Before this commit: robot vacuumcleaner, 5 links, 4 joints
Links:
- removed link base_link
- link base_footprint: mass None -> 2; geometry collision cylinder length=0.04 radius=0.2; collision sphere radius=0.033
Joints:
- removed joint base_joint
- joint base_scan_joint: parent base_link -> base_footprint
- joint joint_left_wheel: parent base_link -> base_footprint
- joint joint_right_wheel: parent base_link -> base_footprint
