Commit message: Model ported to xacro i.s.o urdf. Done to make body radius an argument of the model for experimenting with different radius. radius not correct in movebase YAML files

File: config/vacuumcleaner_model/model.xacro (robot description, xacro)
@@ -1,4 +1,41 @@
-<?xml version="1.0" encoding="UTF-8"?>
-<robot name="vacuumcleaner">
+<robot name="vacuumcleaner" xmlns:xacro="http://wiki.ros.org/xacro">
+  <xacro:property name="body_height" value="0.04"/>
+  <xacro:arg name="body_radius" default="0.2" />
+  <xacro:macro name="wheel" params="suffix radius xoffset yoffset zoffset">
+    <link name="link_${suffix}_wheel">
+      <inertial>
+        <mass value="0.1" />
+        <origin rpy="0 1.5707 1.5707" xyz="0 0 0" />
+        <inertia ixx="2.9925e-5" ixy="0" ixz="0" iyy="2.9925e-5" iyz="0" izz="5.4450e-5" />
+      </inertial>
+      <collision name="link_right_wheel_collision">
+        <origin rpy="0 1.5707 1.5707" xyz="0 0 0" />
+        <geometry>
+          <cylinder length="0.018" radius="${radius}" />
+        </geometry>
+      </collision>
+      <visual name="link_right_wheel_visual">
+        <origin rpy="0 1.5707 1.5707" xyz="0 0 0" />
+        <geometry>
+          <cylinder length="0.018" radius="${radius}" />
+        </geometry>
+      </visual>
+    </link>
+    <gazebo reference="link_${suffix}_wheel">
+       <mu1>100000</mu1>
+       <mu2>100000</mu2>
+       <kp>1e5</kp>
+       <material>Gazebo/Black</material>
+    </gazebo>
+    <joint name="joint_${suffix}_wheel" type="continuous">
+       <origin rpy="0 0 0" xyz="${xoffset} ${yoffset} ${zoffset}" />
+       <child link="link_${suffix}_wheel" />
+       <parent link="base_footprint" />
+       <axis rpy="0 0 0" xyz="0 1 0" />
+       <limit effort="10000" velocity="1000" />
+    </joint>
+  </xacro:macro>
+  <xacro:wheel suffix="left" radius="0.033" xoffset="-0.02" yoffset="${$(arg body_radius) - 0.01}" zoffset="-0.054"/>
+  <xacro:wheel suffix="right" radius="0.033" xoffset="-0.02" yoffset="${-$(arg body_radius) + 0.01}" zoffset="-0.054"/>
   <link name="base_footprint">
     <inertial>
@@ -8,14 +45,14 @@
     <visual>
       <geometry>
-        <cylinder length="0.04" radius="0.2" />
+	      <cylinder length="${body_height}" radius="$(arg body_radius)" />
       </geometry>
     </visual>
     <collision>
       <geometry>
-        <cylinder length="0.04" radius="0.2" />
+	      <cylinder length="${body_height}" radius="$(arg body_radius)" />
       </geometry>
     </collision>
     <collision name="caster_front_collision">
-      <origin rpy="0 0 0" xyz="0.15 0 -0.054" />
+      <origin rpy="0 0 0" xyz="${$(arg body_radius)-0.03} 0 -0.054" />
       <geometry>
         <sphere radius="0.033" />
@@ -23,5 +60,5 @@
     </collision>
     <visual name="caster_front_visual">
-      <origin rpy="0 0 0" xyz="0.15 0 -0.054" />
+      <origin rpy="0 0 0" xyz="${$(arg body_radius) - 0.03} 0 -0.054" />
       <geometry>
         <sphere radius="0.033" />
@@ -29,70 +66,6 @@
     </visual>
   </link>
-  <link name="link_right_wheel">
-    <inertial>
-      <mass value="0.1" />
-      <origin rpy="0 1.5707 1.5707" xyz="0 0 0" />
-      <inertia ixx="2.9925e-5" ixy="0" ixz="0" iyy="2.9925e-5" iyz="0" izz="5.4450e-5" />
-    </inertial>
-    <collision name="link_right_wheel_collision">
-      <origin rpy="0 1.5707 1.5707" xyz="0 0 0" />
-      <geometry>
-        <cylinder length="0.018" radius="0.033" />
-      </geometry>
-    </collision>
-    <visual name="link_right_wheel_visual">
-      <origin rpy="0 1.5707 1.5707" xyz="0 0 0" />
-      <geometry>
-        <cylinder length="0.018" radius="0.033" />
-      </geometry>
-    </visual>
-  </link>
-  <gazebo reference="link_right_wheel">
-    <mu1>100000</mu1>
-    <mu2>100000</mu2>
-    <kp>1e5</kp>
-    <material>Gazebo/Black</material>
-  </gazebo>
-  <link name="link_left_wheel">
-    <inertial>
-      <mass value="0.1" />
-      <origin rpy="0 1.5707 1.5707" xyz="0 0 0" />
-      <inertia ixx="2.9925e-5" ixy="0" ixz="0" iyy="2.9925e-5" iyz="0" izz="5.4450e-5" />
-    </inertial>
-    <collision name="link_left_wheel_collision">
-      <origin rpy="0 1.5707 1.5707" xyz="0 0 0" />
-      <geometry>
-        <cylinder length="0.018" radius="0.033" />
-      </geometry>
-    </collision>
-    <visual name="link_left_wheel_visual">
-      <origin rpy="0 1.5707 1.5707" xyz="0 0 0" />
-      <geometry>
-        <cylinder length="0.018" radius="0.033" />
-      </geometry>
-    </visual>
-  </link>
-  <gazebo reference="link_left_wheel">
-    <mu1>100000</mu1>
-    <mu2>100000</mu2>
-    <kp>1e5</kp>
-    <material>Gazebo/Black</material>
-  </gazebo>
-  <joint name="joint_right_wheel" type="continuous">
-    <origin rpy="0 0 0" xyz="-0.02 -0.10 -0.054" />
-    <child link="link_right_wheel" />
-    <parent link="base_footprint" />
-    <axis rpy="0 0 0" xyz="0 1 0" />
-    <limit effort="10000" velocity="1000" />
-  </joint>
-  <joint name="joint_left_wheel" type="continuous">
-    <origin rpy="0 0 0" xyz="-0.02 0.10 -0.054" />
-    <child link="link_left_wheel" />
-    <parent link="base_footprint" />
-    <axis rpy="0 0 0" xyz="0 1 0" />
-    <limit effort="10000" velocity="1000" />
-  </joint>
   <gazebo>
-    <plugin name="differential_drive" filename="libgazebo_ros_diff_drive.so">
+   <plugin name="differential_drive" filename="libgazebo_ros_diff_drive.so">
       <rosDebugLevel>na</rosDebugLevel>
       <updateRate>30</updateRate>

Commit message: costmap & gmapper published map now take into account radius parameter inertia of disk is now xacro macro

File: config/vacuumcleaner_model/model.xacro (robot description, xacro)
@@ -1,13 +1,22 @@
 <robot name="vacuumcleaner" xmlns:xacro="http://wiki.ros.org/xacro">
+  <xacro:macro name="inertial_disk" params="mass radius height">
+    <inertial>
+      <origin rpy="0 1.5707 1.5707" xyz="0 0 0" />
+      <mass value="${mass}" />
+      <inertia
+        ixx="${1/12 * mass * (3* radius * radius + height * height)}"
+        ixy="0"
+        ixz="0"
+        iyy="${1/12 * mass * (3* radius * radius + height * height)}"
+        iyz="0"
+        izz="${1/2 * mass * radius * radius}" />
+    </inertial>
+  </xacro:macro>
   <xacro:property name="body_height" value="0.04"/>
   <xacro:arg name="body_radius" default="0.2" />
   <xacro:macro name="wheel" params="suffix radius xoffset yoffset zoffset">
     <link name="link_${suffix}_wheel">
-      <inertial>
-        <mass value="0.1" />
-        <origin rpy="0 1.5707 1.5707" xyz="0 0 0" />
-        <inertia ixx="2.9925e-5" ixy="0" ixz="0" iyy="2.9925e-5" iyz="0" izz="5.4450e-5" />
-      </inertial>
-      <collision name="link_right_wheel_collision">
+     <xacro:inertial_disk mass="0.1" radius="${radius}" height="0.018" />
+     <collision name="link_right_wheel_collision">
         <origin rpy="0 1.5707 1.5707" xyz="0 0 0" />
         <geometry>
@@ -39,8 +48,5 @@
   <xacro:wheel suffix="right" radius="0.033" xoffset="-0.02" yoffset="${-$(arg body_radius) + 0.01}" zoffset="-0.054"/>
   <link name="base_footprint">
-    <inertial>
-      <mass value="2" />
-      <inertia ixx="0.02067" ixy="0" ixz="0" iyy="0.020267" iyz="0" izz="0.04" />
-    </inertial>
+    <xacro:inertial_disk mass="2" radius="$(arg body_radius)" height="${body_height}" />
     <visual>
       <geometry>

Commit message: Fix inertia matrix issue on rotated disks

File: config/vacuumcleaner_model/model.xacro (robot description, xacro)
@@ -1,6 +1,6 @@
 <robot name="vacuumcleaner" xmlns:xacro="http://wiki.ros.org/xacro">
-  <xacro:macro name="inertial_disk" params="mass radius height">
+  <xacro:macro name="inertial_disk" params="mass radius height orientation">
     <inertial>
-      <origin rpy="0 1.5707 1.5707" xyz="0 0 0" />
+      <origin rpy="${orientation}" xyz="0 0 0" />
       <mass value="${mass}" />
       <inertia
@@ -16,8 +16,8 @@
   <xacro:arg name="body_radius" default="0.2" />
   <xacro:macro name="wheel" params="suffix radius xoffset yoffset zoffset">
-    <link name="link_${suffix}_wheel">
-     <xacro:inertial_disk mass="0.1" radius="${radius}" height="0.018" />
+     <link name="link_${suffix}_wheel">
+     <xacro:inertial_disk mass="0.1" radius="${radius}" height="0.018" orientation="0 1.5757 1.5757"/>
      <collision name="link_right_wheel_collision">
-        <origin rpy="0 1.5707 1.5707" xyz="0 0 0" />
+        <origin rpy="0 1.5757 1.5757" xyz="0 0 0" />
         <geometry>
           <cylinder length="0.018" radius="${radius}" />
@@ -25,5 +25,5 @@
       </collision>
       <visual name="link_right_wheel_visual">
-        <origin rpy="0 1.5707 1.5707" xyz="0 0 0" />
+        <origin rpy="0 1.5757 1.5757" xyz="0 0 0" />
         <geometry>
           <cylinder length="0.018" radius="${radius}" />
@@ -45,8 +45,8 @@
     </joint>
   </xacro:macro>
-  <xacro:wheel suffix="left" radius="0.033" xoffset="-0.02" yoffset="${$(arg body_radius) - 0.01}" zoffset="-0.054"/>
-  <xacro:wheel suffix="right" radius="0.033" xoffset="-0.02" yoffset="${-$(arg body_radius) + 0.01}" zoffset="-0.054"/>
+  <xacro:wheel suffix="left" radius="0.033" xoffset="-0.01" yoffset="${($(arg body_radius)-0.16)}" zoffset="-0.054"/>
+  <xacro:wheel suffix="right" radius="0.033" xoffset="-0.01" yoffset="${-($(arg body_radius)-0.16)}" zoffset="-0.054"/>
   <link name="base_footprint">
-    <xacro:inertial_disk mass="2" radius="$(arg body_radius)" height="${body_height}" />
+    <xacro:inertial_disk mass="2" radius="$(arg body_radius)" height="${body_height}" orientation="0 0 0"/>
     <visual>
       <geometry>
@@ -78,8 +78,8 @@
       <leftJoint>joint_left_wheel</leftJoint>
       <rightJoint>joint_right_wheel</rightJoint>
-      <wheelSeparation>0.2</wheelSeparation>
+      <wheelSeparation>${ $(arg body_radius)*2 - 0.16*2}</wheelSeparation>
       <wheelDiameter>0.066</wheelDiameter>
       <wheelTorque>20</wheelTorque>
-      <wheelAcceleration>1</wheelAcceleration>
+      <wheelAcceleration>0.1</wheelAcceleration>
       <commandTopic>/cmd_vel</commandTopic>
       <publishOdom>true</publishOdom>
@@ -107,8 +107,5 @@
       </geometry>
     </collision>
-    <inertial>
-      <mass value="0.1" />
-      <inertia ixx="0.0001" ixy="0" ixz="0" iyy="0.0001" iyz="0" izz="0.0001" />
-    </inertial>
+    <xacro:inertial_disk mass="0.001" radius="0.05" height="0.018" orientation="0 0 0"/>
   </link>
   <joint name="base_scan_joint" type="fixed">

Commit message: Use realistic weight for wheels & body; robot tipping over

File: config/vacuumcleaner_model/model.xacro (robot description, xacro)
@@ -1,5 +1,10 @@
 <robot name="vacuumcleaner" xmlns:xacro="http://wiki.ros.org/xacro">
+  <!-- Radius of center disk (meters) -->
+  <xacro:arg name="body_radius" default="0.1"/>
+  <!-- Height of center disk (meters)-->
+  <xacro:property name="body_height" value="0.04"/>
   <xacro:macro name="inertial_disk" params="mass radius height orientation">
     <inertial>
+      <debug mass="${mass}" radius="${radius}" height="${height}" />
       <origin rpy="${orientation}" xyz="0 0 0" />
       <mass value="${mass}" />
@@ -13,10 +18,8 @@
     </inertial>
   </xacro:macro>
-  <xacro:property name="body_height" value="0.04"/>
-  <xacro:arg name="body_radius" default="0.2" />
   <xacro:macro name="wheel" params="suffix radius xoffset yoffset zoffset">
      <link name="link_${suffix}_wheel">
-     <xacro:inertial_disk mass="0.1" radius="${radius}" height="0.018" orientation="0 1.5757 1.5757"/>
-     <collision name="link_right_wheel_collision">
+     <xacro:inertial_disk mass="0.250" radius="${radius}" height="0.018" orientation="0 1.5757 1.5757"/>
+     <collision name="link_${suffix}_wheel_collision">
         <origin rpy="0 1.5757 1.5757" xyz="0 0 0" />
         <geometry>
@@ -24,5 +27,5 @@
         </geometry>
       </collision>
-      <visual name="link_right_wheel_visual">
+      <visual name="link_${suffix}_wheel_visual">
         <origin rpy="0 1.5757 1.5757" xyz="0 0 0" />
         <geometry>
@@ -32,6 +35,6 @@
     </link>
     <gazebo reference="link_${suffix}_wheel">
-       <mu1>100000</mu1>
-       <mu2>100000</mu2>
+       <mu1>1000000</mu1>
+       <mu2>1000000</mu2>
        <kp>1e5</kp>
        <material>Gazebo/Black</material>
@@ -42,11 +45,11 @@
        <parent link="base_footprint" />
        <axis rpy="0 0 0" xyz="0 1 0" />
-       <limit effort="10000" velocity="1000" />
+       <!--<limit effort="10000" velocity="1000" />-->
     </joint>
   </xacro:macro>
-  <xacro:wheel suffix="left" radius="0.033" xoffset="-0.01" yoffset="${($(arg body_radius)-0.16)}" zoffset="-0.054"/>
-  <xacro:wheel suffix="right" radius="0.033" xoffset="-0.01" yoffset="${-($(arg body_radius)-0.16)}" zoffset="-0.054"/>
+  <xacro:wheel suffix="left" radius="0.033" xoffset="0" yoffset="${$(arg body_radius)}" zoffset="-0.054"/>
+  <xacro:wheel suffix="right" radius="0.033" xoffset="0" yoffset="${-$(arg body_radius)}" zoffset="-0.054"/>
   <link name="base_footprint">
-    <xacro:inertial_disk mass="2" radius="$(arg body_radius)" height="${body_height}" orientation="0 0 0"/>
+    <xacro:inertial_disk mass="0.800" radius="$(arg body_radius)" height="${body_height}" orientation="0 0 0" />
     <visual>
       <geometry>
@@ -78,8 +81,7 @@
       <leftJoint>joint_left_wheel</leftJoint>
       <rightJoint>joint_right_wheel</rightJoint>
-      <wheelSeparation>${ $(arg body_radius)*2 - 0.16*2}</wheelSeparation>
+      <wheelSeparation>${2*$(arg body_radius)}</wheelSeparation>
       <wheelDiameter>0.066</wheelDiameter>
-      <wheelTorque>20</wheelTorque>
-      <wheelAcceleration>0.1</wheelAcceleration>
+      <wheelTorque>150</wheelTorque>
       <commandTopic>/cmd_vel</commandTopic>
       <publishOdom>true</publishOdom>
@@ -107,5 +109,10 @@
       </geometry>
     </collision>
-    <xacro:inertial_disk mass="0.001" radius="0.05" height="0.018" orientation="0 0 0"/>
+    <inertial>
+      <mass value="0.01" />
+      <inertia  ixx="0.001" ixy="0.0"  ixz="0.0"
+              iyy="0.001"  iyz="0.0"
+              izz="0.001" />
+    </inertial>
   </link>
   <joint name="base_scan_joint" type="fixed">

Commit message: gazebo: Stop sensor in wobbeling in place

File: config/vacuumcleaner_model/model.xacro (robot description, xacro)
@@ -34,10 +34,12 @@
       </visual>
     </link>
+   <!---
     <gazebo reference="link_${suffix}_wheel">
-       <mu1>1000000</mu1>
-       <mu2>1000000</mu2>
-       <kp>1e5</kp>
+       <mu1>1</mu1>
+       <mu2>1</mu2>
+       <kp>1</kp>
        <material>Gazebo/Black</material>
     </gazebo>
+    -->
     <joint name="joint_${suffix}_wheel" type="continuous">
        <origin rpy="0 0 0" xyz="${xoffset} ${yoffset} ${zoffset}" />
@@ -48,6 +50,11 @@
     </joint>
   </xacro:macro>
-  <xacro:wheel suffix="left" radius="0.033" xoffset="0" yoffset="${$(arg body_radius)}" zoffset="-0.054"/>
-  <xacro:wheel suffix="right" radius="0.033" xoffset="0" yoffset="${-$(arg body_radius)}" zoffset="-0.054"/>
+  <xacro:wheel suffix="left" radius="0.033" xoffset="-0.01" yoffset="${$(arg body_radius)}" zoffset="-0.054"/>
+  <xacro:wheel suffix="right" radius="0.033" xoffset="-0.01" yoffset="${-$(arg body_radius)}" zoffset="-0.054"/>
+  <link name="dummy" />
+  <joint name="dummy_joint" type="fixed">
+     <parent link="dummy"/>
+     <child link="base_footprint"/>
+  </joint>
   <link name="base_footprint">
     <xacro:inertial_disk mass="0.800" radius="$(arg body_radius)" height="${body_height}" orientation="0 0 0" />
@@ -83,5 +90,5 @@
       <wheelSeparation>${2*$(arg body_radius)}</wheelSeparation>
       <wheelDiameter>0.066</wheelDiameter>
-      <wheelTorque>150</wheelTorque>
+      <wheelTorque>0.1</wheelTorque>
       <commandTopic>/cmd_vel</commandTopic>
       <publishOdom>true</publishOdom>
@@ -91,4 +98,7 @@
       <odometryFrame>/odom</odometryFrame>
       <robotBaseFrame>/base_footprint</robotBaseFrame>
+      <wheelAcceleration>0</wheelAcceleration>
+      <publishTf>1</publishTf>
+      <publishWheelJointState>false</publishWheelJointState>
     </plugin>
     <plugin name="joint_state_publisher" filename="libgazebo_ros_joint_state_publisher.so">

Commit message: axarco model: fix flip over. By adding friction to front caster. seems to be a bit too much friction tho. Applying force in direction -> X, will make robot wobble.

File: config/vacuumcleaner_model/model.xacro (robot description, xacro)
@@ -4,5 +4,11 @@
   <!-- Height of center disk (meters)-->
   <xacro:property name="body_height" value="0.04"/>
-  <xacro:macro name="inertial_disk" params="mass radius height orientation">
+  <xacro:macro name="sphere_inertia" params="m r">
+    <inertial>
+      <mass value="${m}"/>
+      <inertia ixx="${2.0*m*(r*r)/5.0}" ixy="0.0" ixz="0.0" iyy="${2.0*m*(r*r)/5.0}" iyz="0.0" izz="${2.0*m*(r*r)/5.0}"/>
+    </inertial>
+  </xacro:macro>
+  <xacro:macro name="disk_inertia" params="mass radius height orientation">
     <inertial>
       <debug mass="${mass}" radius="${radius}" height="${height}" />
@@ -20,5 +26,5 @@
   <xacro:macro name="wheel" params="suffix radius xoffset yoffset zoffset">
      <link name="link_${suffix}_wheel">
-     <xacro:inertial_disk mass="0.250" radius="${radius}" height="0.018" orientation="0 1.5757 1.5757"/>
+     <xacro:disk_inertia mass="0.250" radius="${radius}" height="0.018" orientation="0 1.5757 1.5757"/>
      <collision name="link_${suffix}_wheel_collision">
         <origin rpy="0 1.5757 1.5757" xyz="0 0 0" />
@@ -26,5 +32,5 @@
           <cylinder length="0.018" radius="${radius}" />
         </geometry>
-      </collision>
+     </collision>
       <visual name="link_${suffix}_wheel_visual">
         <origin rpy="0 1.5757 1.5757" xyz="0 0 0" />
@@ -34,13 +40,14 @@
       </visual>
     </link>
-   <!---
-    <gazebo reference="link_${suffix}_wheel">
-       <mu1>1</mu1>
-       <mu2>1</mu2>
-       <kp>1</kp>
-       <material>Gazebo/Black</material>
+     <gazebo reference="link_${suffix}_wheel">
+       <kp>1000000.0</kp>
+       <kd>100.0</kd>
+       <mu1>1.5</mu1>
+       <mu2>1.5</mu2>
+       <fdir1>1 0 0</fdir1>
+       <maxVel>1.0</maxVel>
+       <minDepth>0.00</minDepth>
     </gazebo>
-    -->
-    <joint name="joint_${suffix}_wheel" type="continuous">
+   <joint name="joint_${suffix}_wheel" type="continuous">
        <origin rpy="0 0 0" xyz="${xoffset} ${yoffset} ${zoffset}" />
        <child link="link_${suffix}_wheel" />
@@ -50,6 +57,6 @@
     </joint>
   </xacro:macro>
-  <xacro:wheel suffix="left" radius="0.033" xoffset="-0.01" yoffset="${$(arg body_radius)}" zoffset="-0.054"/>
-  <xacro:wheel suffix="right" radius="0.033" xoffset="-0.01" yoffset="${-$(arg body_radius)}" zoffset="-0.054"/>
+  <xacro:wheel suffix="left" radius="0.033" xoffset="0" yoffset="${$(arg body_radius)}" zoffset="-0.054"/>
+  <xacro:wheel suffix="right" radius="0.033" xoffset="0" yoffset="${-$(arg body_radius)}" zoffset="-0.054"/>
   <link name="dummy" />
   <joint name="dummy_joint" type="fixed">
@@ -58,5 +65,5 @@
   </joint>
   <link name="base_footprint">
-    <xacro:inertial_disk mass="0.800" radius="$(arg body_radius)" height="${body_height}" orientation="0 0 0" />
+    <xacro:disk_inertia mass="0.850" radius="$(arg body_radius)" height="${body_height}" orientation="0 0 0" />
     <visual>
       <geometry>
@@ -69,17 +76,36 @@
       </geometry>
     </collision>
-    <collision name="caster_front_collision">
-      <origin rpy="0 0 0" xyz="${$(arg body_radius)-0.03} 0 -0.054" />
+ </link>
+   <link name="caster_wheel">
+    <visual>
+      <origin xyz="0 0 0" rpy="0 0 0"/>
       <geometry>
-        <sphere radius="0.033" />
+        <sphere radius="0.033"/>
+      </geometry>
+    </visual>
+    <collision>
+      <origin xyz="0 0 0" rpy="0 0 0"/>
+      <geometry>
+        <sphere radius="0.033"/>
       </geometry>
     </collision>
-    <visual name="caster_front_visual">
-      <origin rpy="0 0 0" xyz="${$(arg body_radius) - 0.03} 0 -0.054" />
-      <geometry>
-        <sphere radius="0.033" />
-      </geometry>
-    </visual>
+    <xacro:sphere_inertia m="1" r="0.033"/>
   </link>
+     <gazebo reference="caster_wheel">
+       <kp>1000000.0</kp>
+       <kd>100.0</kd>
+       <mu1>1.5</mu1>
+       <mu2>1.5</mu2>
+       <fdir1>1 0 0</fdir1>
+       <maxVel>1.0</maxVel>
+       <minDepth>0.00</minDepth>
+       <material>Gazebo/ZincYellow</material>
+    </gazebo>
+  <joint name="caster_wheel_joint" type="fixed">
+    <axis xyz="0 1 0" rpy="0 0 0" />
+    <parent link="base_footprint"/>
+    <child link="caster_wheel"/>
+    <origin rpy="0 0 0" xyz="${$(arg body_radius)-0.03} 0 -0.054" />
+  </joint>
   <gazebo>
    <plugin name="differential_drive" filename="libgazebo_ros_diff_drive.so">
@@ -90,5 +116,5 @@
       <wheelSeparation>${2*$(arg body_radius)}</wheelSeparation>
       <wheelDiameter>0.066</wheelDiameter>
-      <wheelTorque>0.1</wheelTorque>
+      <!--<wheelTorque>150</wheelTorque>-->
       <commandTopic>/cmd_vel</commandTopic>
       <publishOdom>true</publishOdom>
@@ -102,4 +128,6 @@
       <publishWheelJointState>false</publishWheelJointState>
     </plugin>
+  </gazebo>
+  <gazebo>
     <plugin name="joint_state_publisher" filename="libgazebo_ros_joint_state_publisher.so">
       <updateRate>30</updateRate>
@@ -130,5 +158,4 @@
     <parent link="base_footprint" />
     <origin xyz="0 0 0.051" />
-    <!-- +0.051 iso 0.05 otherwise vision clips into top of robot-->
   </joint>
   <gazebo reference="base_scan">
