Commit message: Wobble fixed; mapping broken due to dummy link

File: config/vacuumcleaner_model/model.xacro (robot description, xacro)
@@ -43,6 +43,6 @@
        <kp>1000000.0</kp>
        <kd>100.0</kd>
-       <mu1>1.5</mu1>
-       <mu2>1.5</mu2>
+       <mu1>1.0</mu1>
+       <mu2>1.0</mu2>
        <fdir1>1 0 0</fdir1>
        <maxVel>1.0</maxVel>
@@ -57,6 +57,6 @@
     </joint>
   </xacro:macro>
-  <xacro:wheel suffix="left" radius="0.033" xoffset="0" yoffset="${$(arg body_radius)}" zoffset="-0.054"/>
-  <xacro:wheel suffix="right" radius="0.033" xoffset="0" yoffset="${-$(arg body_radius)}" zoffset="-0.054"/>
+  <xacro:wheel suffix="left" radius="0.030" xoffset="0" yoffset="${$(arg body_radius)}" zoffset="-0.055"/>
+  <xacro:wheel suffix="right" radius="0.030" xoffset="0" yoffset="${-$(arg body_radius)}" zoffset="-0.055"/>
   <link name="dummy" />
   <joint name="dummy_joint" type="fixed">
@@ -81,5 +81,5 @@
       <origin xyz="0 0 0" rpy="0 0 0"/>
       <geometry>
-        <sphere radius="0.033"/>
+        <sphere radius="0.030"/>
       </geometry>
     </visual>
@@ -87,14 +87,14 @@
       <origin xyz="0 0 0" rpy="0 0 0"/>
       <geometry>
-        <sphere radius="0.033"/>
+        <sphere radius="0.030"/>
       </geometry>
     </collision>
     <xacro:sphere_inertia m="1" r="0.033"/>
   </link>
-     <gazebo reference="caster_wheel">
+  <gazebo reference="caster_wheel">
        <kp>1000000.0</kp>
        <kd>100.0</kd>
-       <mu1>1.5</mu1>
-       <mu2>1.5</mu2>
+       <mu1>0</mu1>
+       <mu2>0</mu2>
        <fdir1>1 0 0</fdir1>
        <maxVel>1.0</maxVel>
@@ -106,5 +106,5 @@
     <parent link="base_footprint"/>
     <child link="caster_wheel"/>
-    <origin rpy="0 0 0" xyz="${$(arg body_radius)-0.03} 0 -0.054" />
+    <origin rpy="0 0 0" xyz="${$(arg body_radius)-0.03} 0 -0.055" />
   </joint>
   <gazebo>
@@ -116,5 +116,5 @@
       <wheelSeparation>${2*$(arg body_radius)}</wheelSeparation>
       <wheelDiameter>0.066</wheelDiameter>
-      <!--<wheelTorque>150</wheelTorque>-->
+      <wheelTorque>5</wheelTorque>
       <commandTopic>/cmd_vel</commandTopic>
       <publishOdom>true</publishOdom>
@@ -124,5 +124,5 @@
       <odometryFrame>/odom</odometryFrame>
       <robotBaseFrame>/base_footprint</robotBaseFrame>
-      <wheelAcceleration>0</wheelAcceleration>
+      <wheelAcceleration>1.0</wheelAcceleration>
       <publishTf>1</publishTf>
       <publishWheelJointState>false</publishWheelJointState>

Commit message: costmap grid size = gmapping resolution * 4, gives good results.

File: config/vacuumcleaner_model/model.xacro (robot description, xacro)
@@ -59,9 +59,9 @@
   <xacro:wheel suffix="left" radius="0.030" xoffset="0" yoffset="${$(arg body_radius)}" zoffset="-0.055"/>
   <xacro:wheel suffix="right" radius="0.030" xoffset="0" yoffset="${-$(arg body_radius)}" zoffset="-0.055"/>
-  <link name="dummy" />
+  <!--<link name="dummy" />
   <joint name="dummy_joint" type="fixed">
      <parent link="dummy"/>
      <child link="base_footprint"/>
-  </joint>
+  </joint>-->
   <link name="base_footprint">
     <xacro:disk_inertia mass="0.850" radius="$(arg body_radius)" height="${body_height}" orientation="0 0 0" />
@@ -125,6 +125,4 @@
       <robotBaseFrame>/base_footprint</robotBaseFrame>
       <wheelAcceleration>1.0</wheelAcceleration>
-      <publishTf>1</publishTf>
-      <publishWheelJointState>false</publishWheelJointState>
     </plugin>
   </gazebo>

Commit message: Fix model issue, where wheel are outside of vacuumcleaner radius causing clips into terrain. Also added front distance scanner

File: config/vacuumcleaner_model/model.xacro (robot description, xacro)
@@ -4,4 +4,5 @@
   <!-- Height of center disk (meters)-->
   <xacro:property name="body_height" value="0.04"/>
+  <xacro:property name="wheel_height" value="0.018" />
   <xacro:macro name="sphere_inertia" params="m r">
     <inertial>
@@ -24,11 +25,11 @@
     </inertial>
   </xacro:macro>
-  <xacro:macro name="wheel" params="suffix radius xoffset yoffset zoffset">
+  <xacro:macro name="wheel" params="suffix radius length xoffset yoffset zoffset">
      <link name="link_${suffix}_wheel">
-     <xacro:disk_inertia mass="0.250" radius="${radius}" height="0.018" orientation="0 1.5757 1.5757"/>
+     <xacro:disk_inertia mass="0.250" radius="${radius}" height="${length}" orientation="0 1.5757 1.5757"/>
      <collision name="link_${suffix}_wheel_collision">
         <origin rpy="0 1.5757 1.5757" xyz="0 0 0" />
         <geometry>
-          <cylinder length="0.018" radius="${radius}" />
+          <cylinder length="${length}" radius="${radius}" />
         </geometry>
      </collision>
@@ -36,5 +37,5 @@
         <origin rpy="0 1.5757 1.5757" xyz="0 0 0" />
         <geometry>
-          <cylinder length="0.018" radius="${radius}" />
+          <cylinder length="${length}" radius="${radius}" />
         </geometry>
       </visual>
@@ -57,6 +58,6 @@
     </joint>
   </xacro:macro>
-  <xacro:wheel suffix="left" radius="0.030" xoffset="0" yoffset="${$(arg body_radius)}" zoffset="-0.055"/>
-  <xacro:wheel suffix="right" radius="0.030" xoffset="0" yoffset="${-$(arg body_radius)}" zoffset="-0.055"/>
+  <xacro:wheel suffix="left" radius="0.030" length="${wheel_height}" xoffset="0" yoffset="${$(arg body_radius)-wheel_height/2}" zoffset="-0.055"/>
+  <xacro:wheel suffix="right" radius="0.030" length="${wheel_height}" xoffset="0" yoffset="${-$(arg body_radius)+wheel_height/2}" zoffset="-0.055"/>
   <!--<link name="dummy" />
   <joint name="dummy_joint" type="fixed">
@@ -183,8 +184,61 @@
       </ray>
       <plugin name="laserscan" filename="libgazebo_ros_laser.so">
-	<topicName>scan</topicName>
-	<frameName>base_scan</frameName>
+	    <topicName>scan</topicName>
+	    <frameName>base_scan</frameName>
       </plugin>
    </sensor>
   </gazebo>
+  <link name="front_scan">
+    <visual>
+      <geometry>
+        <sphere radius="0.001" />
+      </geometry>
+      <material name="black" />
+    </visual>
+    <collision>
+      <geometry>
+        <sphere radius="0.001" />
+      </geometry>
+    </collision>
+    <inertial>
+      <mass value="0.01" />
+      <inertia  ixx="0.001" ixy="0.0"  ixz="0.0" iyy="0.001"  iyz="0.0"  izz="0.001" />
+    </inertial>
+  </link>
+  <joint name="front_scan_joint" type="fixed">
+    <child link="front_scan" />
+    <parent link="base_footprint" />
+    <origin xyz="$(arg body_radius) 0 0" />
+  </joint>
+ <gazebo reference="front_scan">
+    <sensor name="raycaster_front_scan" type="ray">
+      <always_on>true</always_on>
+      <visualize>true</visualize>
+      <update_rate>5</update_rate>
+      <ray>
+        <scan>
+          <horizontal>
+            <samples>1</samples>
+            <resolution>1.000000</resolution>
+            <min_angle>0.000000</min_angle>
+            <max_angle>6.280000</max_angle>
+          </horizontal>
+        </scan>
+        <range>
+          <min>0.120000</min>
+          <max>3.5</max>
+          <resolution>0.015000</resolution>
+        </range>
+        <noise>
+          <type>gaussian</type>
+          <mean>0.0</mean>
+          <stddev>0.01</stddev>
+        </noise>
+      </ray>
+      <plugin name="laserscan" filename="libgazebo_ros_laser.so">
+    	<topicName>distance_scan</topicName>
+	    <frameName>front_scan</frameName>
+      </plugin>
+   </sensor>
+  </gazebo>
 </robot>

Commit message: Add bumper to model; constrain ossciliation timeout to avoid extremely long trying to reach goal when the goal is impossible to reach; also disabled recovery mechanisms

File: config/vacuumcleaner_model/model.xacro (robot description, xacro)
@@ -72,10 +72,25 @@
       </geometry>
     </visual>
-    <collision>
+    <collision name="base_footprint_collision">
       <geometry>
 	      <cylinder length="${body_height}" radius="$(arg body_radius)" />
       </geometry>
     </collision>
- </link>
+  </link>
+  <gazebo reference="base_footprint">
+    <sensor name='bumper_contact' type='contact'>
+      <plugin name="gazebo_ros_bumper_controller" filename="libgazebo_ros_bumper.so">
+        <bumperTopicName>bumper_vals</bumperTopicName>
+        <frameName>map</frameName>
+        <alwaysOn>true</alwaysOn>
+        <updateRate>4.0</updateRate>
+      </plugin>
+      <always_on>true</always_on>
+      <update_rate>4.0</update_rate>
+      <contact>
+        <collision>base_footprint_collision_collision</collision>
+      </contact>
+    </sensor>
+  </gazebo>
    <link name="caster_wheel">
     <visual>
@@ -189,56 +204,3 @@
    </sensor>
   </gazebo>
-  <link name="front_scan">
-    <visual>
-      <geometry>
-        <sphere radius="0.001" />
-      </geometry>
-      <material name="black" />
-    </visual>
-    <collision>
-      <geometry>
-        <sphere radius="0.001" />
-      </geometry>
-    </collision>
-    <inertial>
-      <mass value="0.01" />
-      <inertia  ixx="0.001" ixy="0.0"  ixz="0.0" iyy="0.001"  iyz="0.0"  izz="0.001" />
-    </inertial>
-  </link>
-  <joint name="front_scan_joint" type="fixed">
-    <child link="front_scan" />
-    <parent link="base_footprint" />
-    <origin xyz="$(arg body_radius) 0 0" />
-  </joint>
- <gazebo reference="front_scan">
-    <sensor name="raycaster_front_scan" type="ray">
-      <always_on>true</always_on>
-      <visualize>true</visualize>
-      <update_rate>5</update_rate>
-      <ray>
-        <scan>
-          <horizontal>
-            <samples>1</samples>
-            <resolution>1.000000</resolution>
-            <min_angle>0.000000</min_angle>
-            <max_angle>6.280000</max_angle>
-          </horizontal>
-        </scan>
-        <range>
-          <min>0.120000</min>
-          <max>3.5</max>
-          <resolution>0.015000</resolution>
-        </range>
-        <noise>
-          <type>gaussian</type>
-          <mean>0.0</mean>
-          <stddev>0.01</stddev>
-        </noise>
-      </ray>
-      <plugin name="laserscan" filename="libgazebo_ros_laser.so">
-    	<topicName>distance_scan</topicName>
-	    <frameName>front_scan</frameName>
-      </plugin>
-   </sensor>
-  </gazebo>
 </robot>
