Commit message: Update gazebo_ros_diff_drive to foxy version

File: models/robot.xacro (robot description, xacro)
@@ -53,5 +53,5 @@
        <origin rpy="0 0 0" xyz="${xoffset} ${yoffset} ${zoffset}" />
        <child link="link_${suffix}_wheel" />
-       <parent link="base_footprint" />
+       <parent link="base_link" />
        <axis rpy="0 0 0" xyz="0 1 0" />
        <!--<limit effort="10000" velocity="1000" />-->
@@ -63,7 +63,7 @@
   <joint name="dummy_joint" type="fixed">
      <parent link="dummy"/>
-     <child link="base_footprint"/>
+     <child link="base_link"/>
   </joint>-->
-  <link name="base_footprint">
+  <link name="base_link">
     <xacro:disk_inertia mass="0.850" radius="$(arg body_radius)" height="${body_height}" orientation="0 0 0" />
     <visual>
@@ -72,5 +72,5 @@
       </geometry>
     </visual>
-    <collision name="base_footprint_collision">
+    <collision name="base_link_collision">
       <geometry>
 	      <cylinder length="${body_height}" radius="$(arg body_radius)" />
@@ -79,5 +79,5 @@
   </link>
   <!--
-  <gazebo reference="base_footprint">
+  <gazebo reference="base_link">
     <sensor name='bumper_contact' type='contact'>
       <plugin name="gazebo_ros_bumper_controller" filename="libgazebo_ros_bumper.so">
@@ -90,5 +90,5 @@
       <update_rate>4.0</update_rate>
       <contact>
-        <collision>base_footprint_collision_collision</collision>
+        <collision>base_link_collision_collision</collision>
       </contact>
     </sensor>
@@ -122,10 +122,10 @@
   <joint name="caster_wheel_joint" type="fixed">
     <axis xyz="0 1 0" rpy="0 0 0" />
-    <parent link="base_footprint"/>
+    <parent link="base_link"/>
     <child link="caster_wheel"/>
     <origin rpy="0 0 0" xyz="${$(arg body_radius)-0.03} 0 -0.055" />
   </joint>
   <gazebo>
-   <plugin name="differential_drive" filename="libgazebo_ros_diff_drive.so">
+   <plugin name="differential_drive_controller" filename="libgazebo_ros_diff_drive.so">
       <ros_debug_level>na</ros_debug_level>
       <update_rate>30</update_rate>
@@ -140,7 +140,7 @@
       <publish_wheel_tf>false</publish_wheel_tf>
       <odometry_topic>/odom</odometry_topic>
+      <wheel_acceleration>1.0</wheel_acceleration>
       <odometry_frame>/odom</odometry_frame>
-      <robotBase_frame>/base_footprint</robotBase_frame>
-      <wheel_acceleration>1.0</wheel_acceleration>
+      <robot_base_frame>/base_link</robot_base_frame>
     </plugin>
   </gazebo>
@@ -176,5 +176,5 @@
   <joint name="base_scan_joint" type="fixed">
     <child link="base_scan" />
-    <parent link="base_footprint" />
+    <parent link="base_link" />
     <origin xyz="0 0 0.051" />
   </joint>

Commit message: rename base_scan to map

File: models/robot.xacro (robot description, xacro)
@@ -155,5 +155,5 @@
     </plugin>
   </gazebo>
-  <link name="base_scan">
+  <link name="map">
     <visual>
       <geometry>
@@ -174,10 +174,10 @@
     </inertial>
   </link>
-  <joint name="base_scan_joint" type="fixed">
-    <child link="base_scan" />
+  <joint name="map_joint" type="fixed">
+    <child link="map" />
     <parent link="base_link" />
     <origin xyz="0 0 0.051" />
   </joint>
-  <gazebo reference="base_scan">
+  <gazebo reference="map">
     <sensor name="raycaster" type="ray">
       <always_on>true</always_on>
@@ -209,5 +209,5 @@
         </ros>
         <output_type>sensor_msgs/LaserScan</output_type>
-        <frame_name>base_scan</frame_name>
+        <frame_name>map</frame_name>
       </plugin>
    </sensor>

Commit message: Fix tf2 odom tree issue

File: models/robot.xacro (robot description, xacro)
@@ -60,7 +60,7 @@
   <xacro:wheel suffix="left" radius="0.030" length="${wheel_height}" xoffset="0" yoffset="${$(arg body_radius)-wheel_height/2}" zoffset="-0.055"/>
   <xacro:wheel suffix="right" radius="0.030" length="${wheel_height}" xoffset="0" yoffset="${-$(arg body_radius)+wheel_height/2}" zoffset="-0.055"/>
-  <!--<link name="dummy" />
-  <joint name="dummy_joint" type="fixed">
-     <parent link="dummy"/>
+  <!--<link name="base_footprint" />
+  <joint name="base_footprint_joint" type="fixed">
+     <parent link="base_footprint"/>
      <child link="base_link"/>
   </joint>-->
@@ -127,5 +127,5 @@
   </joint>
   <gazebo>
-   <plugin name="differential_drive_controller" filename="libgazebo_ros_diff_drive.so">
+   <plugin name="gazebo_ros_diff_drive" filename="libgazebo_ros_diff_drive.so">
       <ros_debug_level>na</ros_debug_level>
       <update_rate>30</update_rate>
@@ -139,8 +139,8 @@
       <publish_odom_tf>true</publish_odom_tf>
       <publish_wheel_tf>false</publish_wheel_tf>
-      <odometry_topic>/odom</odometry_topic>
+      <odometry_topic>odom</odometry_topic>
       <wheel_acceleration>1.0</wheel_acceleration>
-      <odometry_frame>/odom</odometry_frame>
-      <robot_base_frame>/base_link</robot_base_frame>
+      <odometry_frame>odom</odometry_frame>
+      <robot_base_frame>base_link</robot_base_frame>
     </plugin>
   </gazebo>

Commit message: change map linke name to scanner

File: models/robot.xacro (robot description, xacro)
@@ -60,9 +60,9 @@
   <xacro:wheel suffix="left" radius="0.030" length="${wheel_height}" xoffset="0" yoffset="${$(arg body_radius)-wheel_height/2}" zoffset="-0.055"/>
   <xacro:wheel suffix="right" radius="0.030" length="${wheel_height}" xoffset="0" yoffset="${-$(arg body_radius)+wheel_height/2}" zoffset="-0.055"/>
-  <!--<link name="base_footprint" />
-  <joint name="base_footprint_joint" type="fixed">
-     <parent link="base_footprint"/>
+  <link name="virtual_base_link" />
+  <joint name="virtual_base_link_joint" type="fixed">
+     <parent link="virtual_base_link"/>
      <child link="base_link"/>
-  </joint>-->
+  </joint>
   <link name="base_link">
     <xacro:disk_inertia mass="0.850" radius="$(arg body_radius)" height="${body_height}" orientation="0 0 0" />
@@ -142,5 +142,5 @@
       <wheel_acceleration>1.0</wheel_acceleration>
       <odometry_frame>odom</odometry_frame>
-      <robot_base_frame>base_link</robot_base_frame>
+      <robot_base_frame>virtual_base_link</robot_base_frame>
     </plugin>
   </gazebo>
@@ -155,5 +155,5 @@
     </plugin>
   </gazebo>
-  <link name="map">
+  <link name="scan_link">
     <visual>
       <geometry>
@@ -174,10 +174,10 @@
     </inertial>
   </link>
-  <joint name="map_joint" type="fixed">
-    <child link="map" />
+  <joint name="scan_link_joint" type="fixed">
+    <child link="scan_link" />
     <parent link="base_link" />
     <origin xyz="0 0 0.051" />
   </joint>
-  <gazebo reference="map">
+  <gazebo reference="scan_link">
     <sensor name="raycaster" type="ray">
       <always_on>true</always_on>
@@ -209,5 +209,5 @@
         </ros>
         <output_type>sensor_msgs/LaserScan</output_type>
-        <frame_name>map</frame_name>
+        <frame_name>scan_link</frame_name>
       </plugin>
    </sensor>
